Commit message: z axiz to gazebo and rviz

File: scara_arm_description/urdf/scara_arm.xacro (robot description, xacro)
@@ -4,4 +4,10 @@
 <xacro:include filename="$(find scara_arm_description)/urdf/scara_arm.trans" />
 <xacro:include filename="$(find scara_arm_description)/urdf/scara_arm.gazebo" />
+<link name="world" />
+    <joint name="world_joint" type="fixed">
+        <origin rpy="0 0 0" xyz="0 0 0.25" />
+        <parent link="world" />
+        <child link="base_link" />
+    </joint>
 <link name="base_link">
   <inertial>

Commit message: updated xacro to real life robot

File: scara_arm_description/urdf/scara_arm.xacro (robot description, xacro)
@@ -115,5 +115,5 @@
   <child link="link_01_1"/>
   <axis xyz="0.0 -0.0 1.0"/>
-  <limit upper="1.570796" lower="-1.570796" effort="100" velocity="100"/>
+  <limit upper="1.71042" lower="-1.43117" effort="100" velocity="100"/>
 </joint>
 <joint name="link_02_joint" type="revolute">
@@ -122,5 +122,5 @@
   <child link="link_02_1"/>
   <axis xyz="0.0 0.0 1.0"/>
-  <limit upper="1.570796" lower="-1.570796" effort="100" velocity="100"/>
+  <limit upper="1.43117" lower="-1.71042" effort="100" velocity="100"/>
 </joint>
 <joint name="link_03_joint" type="prismatic">
