Commit message: xacro for vacuum gripper added

File: scara_arm_description/urdf/scara_arm_vacuum_gripper.xacro (robot description, xacro)
@@ -1,8 +1,8 @@
 <?xml version="1.0" ?>
-<robot name="scara_arm_two_finger_gripper" xmlns:xacro="http://www.ros.org/wiki/xacro">
+<robot name="scara_arm_vacuum_gripper" xmlns:xacro="http://www.ros.org/wiki/xacro">
 <xacro:include filename="$(find scara_arm_description)/urdf/scara_arm.xacro" />
-<xacro:include filename="$(find two_finger_gripper_description)/urdf/two_finger_gripper.xacro" />
+<xacro:include filename="$(find vacuum_gripper_description)/urdf/vacuum_gripper.xacro" />
 <joint name="gripper_attach" type="fixed">
-  <origin xyz="0 0 0" rpy="0 1.5708 0"/>
+  <origin xyz="0 0 0" rpy="0 0 0"/>
   <parent link="link_04_1"/>
   <child link="gripper_base_link"/>
