Commit message: Init

File: scara_arm_config/config/gazebo_scara_arm.urdf (robot description, URDF)
Before this commit: robot scara_arm, 5 links, 4 joints
Links:
- added link world
Joints:
- added joint world_joint: type fixed, parent world, child base_link, origin xyz=0 0 0.25 rpy=0 0 0
- joint link_01_joint: limit lower=-1.570796 upper=1.570796 effort=100 velocity=100 -> lower=-1.43117 upper=1.71042 effort=100 velocity=100
- joint link_02_joint: limit lower=-1.570796 upper=1.570796 effort=100 velocity=100 -> lower=-1.71042 upper=1.43117 effort=100 velocity=100

Commit message: Suction Gripper DONE

File: scara_arm_config/config/gazebo_scara_arm.urdf (robot description, URDF)
Before this commit: robot scara_arm, 6 links, 5 joints
Links:
- added link gripper_base_link, mass 0.8034775156193473; collision mesh filename=package://scara_arm_description/meshes/suction_gripper/grip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 scale=0.001 0.001 0.001; visual mesh filename=package://scara_arm_description/meshes/suction_gripper/grip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 scale=0.001 0.001 0.001
- added link gripper_link_1, mass 0.002457048975733048; collision mesh filename=package://scara_arm_description/meshes/suction_gripper/grip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 scale=0.001 0.001 0.001; visual mesh filename=package://scara_arm_description/meshes/suction_gripper/grip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 scale=0.001 0.001 0.001
Joints:
- added joint gripper_attach: type fixed, parent link_04_1, child gripper_base_link, origin xyz=0 0 0 rpy=0 0 0
- added joint gripper_joint: type prismatic, parent gripper_base_link, child gripper_link_1, origin xyz=0.000371 2.9e-05 -0.0505 rpy=0 0 0, axis -0.0 -0.0 -1.0, limit lower=0.0 upper=0.02 effort=100 velocity=100

Commit message: scara_arm_config restored for only arm

File: scara_arm_config/config/gazebo_scara_arm.urdf (robot description, URDF)
Before this commit: robot scara_arm, 8 links, 7 joints
Links:
- removed link gripper_base_link
- removed link gripper_link_1
Joints:
- removed joint gripper_attach
- removed joint gripper_joint
